Commit message: fix: remove gripper collision geometry to fix MoveIt START_STATE_IN_COLLISION

File: src/ur5_simulation/urdf/simple_gripper.xacro (robot description, xacro)
@@ -9,8 +9,4 @@
         <material name="gripper_gray"><color rgba="0.5 0.5 0.5 1"/></material>
       </visual>
-      <collision>
-        <origin xyz="0 0 0.01" rpy="0 0 0"/>
-        <geometry><box size="0.06 0.06 0.02"/></geometry>
-      </collision>
       <inertial>
         <mass value="0.3"/>
@@ -31,8 +27,4 @@
         <material name="gripper_dark"><color rgba="0.2 0.2 0.2 1"/></material>
       </visual>
-      <collision>
-        <origin xyz="0 0.006 -0.02" rpy="0 0 0"/>
-        <geometry><box size="0.012 0.012 0.04"/></geometry>
-      </collision>
       <inertial>
         <mass value="0.05"/>
@@ -55,8 +47,4 @@
         <material name="gripper_dark"><color rgba="0.2 0.2 0.2 1"/></material>
       </visual>
-      <collision>
-        <origin xyz="0 -0.006 -0.02" rpy="0 0 0"/>
-        <geometry><box size="0.012 0.012 0.04"/></geometry>
-      </collision>
       <inertial>
         <mass value="0.05"/>

Commit message: fix: replace mimic joint with dual command interfaces for Gazebo Harmonic

File: src/ur5_simulation/urdf/simple_gripper.xacro (robot description, xacro)
@@ -59,7 +59,6 @@
       <axis xyz="0 -1 0"/>
       <limit lower="0.0" upper="0.04" effort="50.0" velocity="0.5"/>
-      <mimic joint="${prefix}left_finger_joint" multiplier="1" offset="0"/>
     </joint>
-    <!-- ros2_control interface — only left_finger_joint is commanded -->
+    <!-- ros2_control interface — both fingers commanded directly (no mimic support in Gazebo Harmonic) -->
     <ros2_control name="${prefix}GripperSystem" type="system">
       <hardware>
@@ -76,4 +75,8 @@
       </joint>
       <joint name="${prefix}right_finger_joint">
+        <command_interface name="position">
+          <param name="min">0</param>
+          <param name="max">0.04</param>
+        </command_interface>
         <state_interface name="position"/>
         <state_interface name="velocity"/>
